Commit message: added rock_box

File: models/prismatic_box/model.urdf (robot description, URDF)
Before this commit: robot prismatic_box, 4 links, 3 joints
Links:
- removed link prismatic_box
- added link slide_box, mass 10000; collision box size=18 12 0.5; visual box size=18 12 0.5
Joints:
- removed joint prismatic_box_joint
- added joint slide_box_joint: type fixed, parent world_box, child slide_box, origin xyz=0 0 1.25 rpy=0 0 0
- joint box_joint: parent prismatic_box -> slide_box

Commit message: fixed linear space sampling and shake table

File: models/prismatic_box/model.urdf (robot description, URDF)
Before this commit: robot prismatic_box, 4 links, 3 joints
Links:
- link slide_box: mass 10000 -> 500000; geometry collision box size=50 12 0.5; visual box size=50 12 0.5
- link world_box: mass 50000 -> 5000000; geometry collision box size=50 14 2; visual box size=50 14 2
Joints:
- joint box_joint: limit lower=-4 upper=4 effort=1000000 velocity=20 -> lower=-25 upper=25 effort=10000000 velocity=200
