Commit message: modified shake table

File: models/prismatic_large_box/model_cube.urdf (robot description, URDF)
Before this commit: robot prismatic_box, 4 links, 3 joints
Links:
- link box: mass 15000 -> 10000; geometry collision mesh filename=package://gazebo_sim_models/models/cube/cube.dae; visual mesh filename=package://gazebo_sim_models/models/cube/cube.dae
