Commit message: fragility anisotripy from niche

File: models/granite_dell/model.urdf (robot description, URDF)
Before this commit: robot prismatic_box, 4 links, 3 joints
Links:
- link box: geometry collision mesh filename=package://gazebo_sim_models/models/granite_dell/granite_del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; visual mesh filename=package://gazebo_sim_models/models/granite_dell/granite_del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
